File: Elettronica/PCB/PCB.brd (EAGLE design)
At the start: 177.6 x 159 mm, 60 parts, among them IC1 7805TV, J2 455-1750-1-ND, SW2 EC12E_SW

Commit message: Elettronica modifiche
Routing:
- net 12V: track 293.7 -> 296.2 mm
Changed lines of the file:
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@@
 <?xml version="1.0" encoding="utf-8"?>
 <!DOCTYPE eagle SYSTEM "eagle.dtd">
-<eagle version="9.3.1">
+<eagle version="9.2.2">
 <drawing>
 <settings>
@@
 <contactref element="X1" pad="1"/>
 <contactref element="X3" pad="1"/>
-<wire x1="14.653259375" y1="99.118421875" x2="24.813259375" y2="109.278421875" width="2" layer="16"/>
-<wire x1="24.813259375" y1="109.278421875" x2="24.813259375" y2="155.709621875" width="2" layer="16"/>
+<wire x1="24.813259375" y1="105.036621875" x2="18.895059375" y2="99.118421875" width="2" layer="16"/>
+<wire x1="14.653259375" y1="99.118421875" x2="18.895059375" y2="99.118421875" width="2" layer="16"/>
+<wire x1="24.813259375" y1="105.036621875" x2="24.813259375" y2="155.709621875" width="2" layer="16"/>
 <wire x1="31.696659375" y1="162.593021875" x2="24.813259375" y2="155.709621875" width="2" layer="16"/>
 <wire x1="87.068659375" y1="158.783021875" x2="83.258659375" y2="162.593021875" width="2" layer="16"/>
@@
 <contactref element="R3" pad="2"/>
 <contactref element="B1" pad="9"/>
-<wire x1="148.257259375" y1="96.553021875" x2="148.257259375" y2="106.459021875" width="0.6096" layer="1"/>
-<wire x1="148.257259375" y1="106.459021875" x2="149.273259375" y2="107.475021875" width="0.6096" layer="1"/>
-<wire x1="149.273259375" y1="107.475021875" x2="159.433259375" y2="107.475021875" width="0.6096" layer="1"/>
-<wire x1="159.433259375" y1="107.475021875" x2="160.703259375" y2="108.745021875" width="0.6096" layer="1"/>
-<wire x1="160.703259375" y1="108.745021875" x2="160.703259375" y2="123.477021875" width="0.6096" layer="1"/>
+<wire x1="148.257259375" y1="96.553021875" x2="148.257259375" y2="108.135421875" width="0.6096" layer="1"/>
+<wire x1="148.257259375" y1="108.135421875" x2="150.009859375" y2="109.888021875" width="0.6096" layer="1"/>
+<wire x1="150.009859375" y1="109.888021875" x2="160.703259375" y2="109.888021875" width="0.6096" layer="1"/>
+<wire x1="160.703259375" y1="109.888021875" x2="160.703259375" y2="123.477021875" width="0.6096" layer="1"/>
 <wire x1="160.703259375" y1="123.477021875" x2="161.465259375" y2="124.239021875" width="0.6096" layer="1"/>
 <wire x1="161.465259375" y1="124.239021875" x2="168.171259375" y2="124.239021875" width="0.6096" layer="1"/>
@@
 <via x="157.655259375" y="140.749021875" extent="1-16" drill="0.55"/>
 <wire x1="157.655259375" y1="140.749021875" x2="157.655259375" y2="120.175021875" width="0.6096" layer="1"/>
-<wire x1="157.655259375" y1="120.175021875" x2="150.797259375" y2="113.317021875" width="0.6096" layer="1"/>
-<wire x1="150.797259375" y1="113.317021875" x2="150.797259375" y2="109.507021875" width="0.6096" layer="1"/>
-<via x="150.797259375" y="109.507021875" extent="1-16" drill="0.508"/>
-<wire x1="150.797259375" y1="109.507021875" x2="150.797259375" y2="105.443021875" width="0.6096" layer="16"/>
+<wire x1="157.655259375" y1="120.175021875" x2="150.848059375" y2="113.367821875" width="0.6096" layer="1"/>
+<wire x1="150.848059375" y1="113.367821875" x2="150.848059375" y2="112.529621875" width="0.6096" layer="1"/>
+<via x="150.848059375" y="112.529621875" extent="1-16" drill="0.508"/>
+<wire x1="150.848059375" y1="112.529621875" x2="150.848059375" y2="105.493821875" width="0.6096" layer="16"/>
+<wire x1="150.797259375" y1="105.443021875" x2="150.848059375" y2="105.493821875" width="0.6096" layer="16"/>
 <via x="150.797259375" y="105.443021875" extent="1-16" drill="0.508"/>
 <wire x1="150.797259375" y1="105.443021875" x2="150.797259375" y2="96.553021875" width="0.6096" layer="1"/>
